File: KiCAD/Dianome.kicad_sch (KiCad schematic)
At the start: 38 parts, among them J1 Screw_Terminal_01x06, J2 USB_C_Receptacle_USB2.0, J3 Conn_01x02_Male, J4 Conn_01x02_Male, J5 Screw_Terminal_01x06, J6 Screw_Terminal_01x01, J7 Screw_Terminal_01x01, Q1 Q_NMOS_DGS, U1 ΜΑΧ17504, U2 LM5060

Commit message: minor layout changes
Other:
- company: (none) -> Tinymovr
- title: (none) -> Dianome Power Distribution Board
- moved on the sheet: J1, J5, J6, J7
